Commit message: Add plugins to 1. control the movement of car using arrow key 2. get data from imu and lidar

File: sentry_gazebo/urdf/test_robot.xacro (robot description, xacro)
@@ -163,45 +163,22 @@
     </inertial>
   </link>
-  <!-- Gazebo plugin settings related -->
-  <gazebo reference="base_link">
-    <material>Gazebo/Orange</material>
-  </gazebo>
-  <gazebo reference="wheel_1">
-    <material>Gazebo/Red</material>
-  </gazebo>
-  <gazebo reference="wheel_2">
-    <material>Gazebo/Black</material>
-  </gazebo>
-  <gazebo reference="wheel_3">
-    <material>Gazebo/Red</material>
-  </gazebo>
-  <gazebo reference="wheel_4">
-    <material>Gazebo/Black</material>
-  </gazebo>
-  <gazebo reference="imu_link">
-    <material>Gazebo/BuildingFrame</material>
-  </gazebo>
-  <gazebo reference="livox_frame">
-    <material>Gazebo/LightBlueLaser</material>
-  </gazebo>
-  <!-- Drive controller plugin-->
+  <!-- Robot Plugins-->
   <!-- https://gazebosim.org/docs/fortress/moving_robot/ -->
   <gazebo>
-    <!-- <plugin name="mecanum_controller" filename="libgazebo_ros_planar_move.so">
-      <robotNamespace>/</robotNamespace>
-        <commandTopic>/A/car0/cmd_vel</commandTopic> -->
-        <!-- <remapping>cmd_vel:=/A/car0/cmd_vel</remapping> -->
-        <!-- <odometryTopic>odom</odometryTopic>
-        <odometryFrame>odom</odometryFrame>
-        <leftFrontJoint>base_to_wheel1</leftFrontJoint>
-        <rightFrontJoint>base_to_wheel2</rightFrontJoint>
-        <leftRearJoint>base_to_wheel3</leftRearJoint>
-        <rightRearJoint>base_to_wheel4</rightRearJoint>
-        <odometryRate>60.0</odometryRate>
-        <robotBaseFrame>base_link</robotBaseFrame>
-    </plugin> -->
-    <plugin
-        filename="libignition-gazebo-diff-drive-system.so"
-        name="ignition::gazebo::systems::DiffDrive">
+    <plugin filename="libignition-gazebo-sensors-system.so"
+            name="ignition::gazebo::systems::Sensors">
+        <render_engine>ogre2</render_engine>
+    </plugin>
+    <plugin filename="libignition-gazebo-user-commands-system.so"
+            name="ignition::gazebo::systems::UserCommands">
+    </plugin>
+    <!--shows the scene in the GUI-->
+    <plugin filename="libignition-gazebo-scene-broadcaster-system.so"
+            name="ignition::gazebo::systems::SceneBroadcaster">
+    </plugin>
+    <!-- DiffDrive plugin -->
+    <!-- can be changed to libignition-gazebo-mecanum-drive-system.so for mecanum drive, there's even a wheel-slip plugin -->
+    <plugin filename="libignition-gazebo-diff-drive-system.so"
+            name="ignition::gazebo::systems::DiffDrive">
         <left_joint>base_to_wheel1</left_joint>
         <left_joint>base_to_wheel2</left_joint>
@@ -213,9 +190,9 @@
         <topic>cmd_vel</topic>
     </plugin>
-    <!-- Moving Forward-->
-    <plugin filename="libignition-gazebo-triggered-publisher-system.so"
-            name="ignition::gazebo::systems::TriggeredPublisher">
-        <input type="ignition.msgs.Int32" topic="/keyboard/keypress">
-            <match field="data">16777235</match> <!-- Up arrow key -->
+    <!-- Moving Forward with Arrow Key Control plugin -->
+    <plugin filename="libignition-gazebo-triggered-publisher-system.so"
+            name="ignition::gazebo::systems::TriggeredPublisher">
+        <input type="ignition.msgs.Int32" topic="/keyboard/keypress">
+            <match field="data">16777235</match>
         </input>
         <output type="ignition.msgs.Twist" topic="/cmd_vel">
@@ -223,9 +200,9 @@
         </output>
     </plugin>
-    <!-- Moving Backward-->
-    <plugin filename="libignition-gazebo-triggered-publisher-system.so"
-            name="ignition::gazebo::systems::TriggeredPublisher">
-        <input type="ignition.msgs.Int32" topic="/keyboard/keypress">
-            <match field="data">16777237</match> <!-- Down arrow key -->
+    <!-- Moving Backward with Arrow Key Control plugin -->
+    <plugin filename="libignition-gazebo-triggered-publisher-system.so"
+            name="ignition::gazebo::systems::TriggeredPublisher">
+        <input type="ignition.msgs.Int32" topic="/keyboard/keypress">
+            <match field="data">16777237</match>
         </input>
         <output type="ignition.msgs.Twist" topic="/cmd_vel">
@@ -233,9 +210,9 @@
         </output>
     </plugin>
-    <!-- Turning Left-->
-    <plugin filename="libignition-gazebo-triggered-publisher-system.so"
-            name="ignition::gazebo::systems::TriggeredPublisher">
-        <input type="ignition.msgs.Int32" topic="/keyboard/keypress">
-            <match field="data">16777234</match> <!-- Left arrow key -->
+    <!-- Turning Left with Arrow Key Control plugin -->
+    <plugin filename="libignition-gazebo-triggered-publisher-system.so"
+            name="ignition::gazebo::systems::TriggeredPublisher">
+        <input type="ignition.msgs.Int32" topic="/keyboard/keypress">
+            <match field="data">16777234</match>
         </input>
         <output type="ignition.msgs.Twist" topic="/cmd_vel">
@@ -243,9 +220,9 @@
         </output>
     </plugin>
-    <!-- Turning Right-->
-    <plugin filename="libignition-gazebo-triggered-publisher-system.so"
-            name="ignition::gazebo::systems::TriggeredPublisher">
-        <input type="ignition.msgs.Int32" topic="/keyboard/keypress">
-            <match field="data">16777236</match> <!-- Right arrow key -->
+    <!-- Turning Right with Arrow Key Control plugin -->
+    <plugin filename="libignition-gazebo-triggered-publisher-system.so"
+            name="ignition::gazebo::systems::TriggeredPublisher">
+        <input type="ignition.msgs.Int32" topic="/keyboard/keypress">
+            <match field="data">16777236</match>
         </input>
         <output type="ignition.msgs.Twist" topic="/cmd_vel">
@@ -253,9 +230,9 @@
         </output>
     </plugin>
-    <!-- Stop-->
-    <plugin filename="libignition-gazebo-triggered-publisher-system.so"
-            name="ignition::gazebo::systems::TriggeredPublisher">
-        <input type="ignition.msgs.Int32" topic="/keyboard/keypress">
-            <match field="data">49</match> <!-- 1 key -->
+    <!-- Stop with Key '1' Control plugin -->
+    <plugin filename="libignition-gazebo-triggered-publisher-system.so"
+            name="ignition::gazebo::systems::TriggeredPublisher">
+        <input type="ignition.msgs.Int32" topic="/keyboard/keypress">
+            <match field="data">49</match>
         </input>
         <output type="ignition.msgs.Twist" topic="/cmd_vel">
@@ -264,11 +241,13 @@
     </plugin>
   </gazebo>
-  <!-- mid360_imu plugin -->
-  <!-- https://github.com/ros-simulation/gazebo_ros_pkgs/wiki/ROS-2-Migration:-IMU-Sensors -->
+  <!-- link plugins -->
+  <!-- there's also an odometry-publish-system plugin for publishing odom topic -->
+  <!-- mid360_imu sensor and its plugin -->
+  <!-- topic name in ign topic -l: /world/default/model/testbot/link/dummy/sensor/mid360_imu/imu -->
   <gazebo reference="imu_link">
     <sensor name="mid360_imu" type="imu">
       <always_on>true</always_on>
       <update_rate>100</update_rate>
-      <plugin name="imu_plugin" filename="libgazebo_ros_imu_sensor.so">
+      <plugin name="ignition::gazebo::systems::Imu" filename="libignition-gazebo-imu-system.so">
         <ros>
           <namespace>/</namespace>
@@ -279,4 +258,29 @@
     </sensor>
   </gazebo>
+  <!-- LiDAR sensor -->
+  <!-- https://gazebosim.org/docs/fortress/sensors/#lidar-sensor -->
+  <!-- topic name in ign topic -l: /world/default/model/testbot/link/dummy/sensor/lidar_sensor/scan -->
+  <gazebo reference="base_link">
+    <sensor type="gpu_ray" name="lidar_sensor">
+      <pose>0 0 0 0 0 0</pose>
+      <visualize>true</visualize>
+      <update_rate>20</update_rate>
+      <ray>
+        <scan>
+          <horizontal>
+            <samples>360</samples>
+            <resolution>1</resolution>
+            <min_angle>-1.5708</min_angle>
+            <max_angle>1.5708</max_angle>
+          </horizontal>
+        </scan>
+        <range>
+          <min>0.2</min>
+          <max>10.0</max>
+          <resolution>0.01</resolution>
+        </range>
+      </ray>
+    </sensor>
+  </gazebo>
   <!-- Livox-Mid360  -->
   <!--<xacro:include filename="$(find ros2_livox_simulation)/urdf/mid360.xacro" />

Commit message: Fixed the jitter issues and integrated our nav stack into the sim. Also cleaned up the workspace by moving extra packages to backups and updated the README with the new build steps.

File: sentry_gazebo/urdf/test_robot.xacro (robot description, xacro)
@@ -14,5 +14,4 @@
   <xacro:arg name="xyz" default="0.12 0.0 0.175" />
   <xacro:arg name="rpy" default="0 0 0" />
-  <link name="dummy"/>
   <link name="base_link">
     <visual>
@@ -33,8 +32,4 @@
     <xacro:default_inertial mass="8.2"/>
   </link>
-  <joint name="dummy_joint" type="fixed">
-     <parent link="dummy"/>
-     <child link="base_link"/>
-  </joint>
   <link name="wheel_1">
     <visual>
@@ -181,12 +176,16 @@
     <plugin filename="libignition-gazebo-diff-drive-system.so"
             name="ignition::gazebo::systems::DiffDrive">
-        <left_joint>base_to_wheel1</left_joint>
-        <left_joint>base_to_wheel2</left_joint>
+        <left_joint>base_to_wheel1</left_joint> <left_joint>base_to_wheel2</left_joint>
         <right_joint>base_to_wheel3</right_joint>
         <right_joint>base_to_wheel4</right_joint>
         <wheel_separation>1.2</wheel_separation>
         <wheel_radius>${radius_wheel}</wheel_radius>
-        <odom_publish_frequency>1</odom_publish_frequency>
+        <odom_publish_frequency>50</odom_publish_frequency>
+        <use_sim_time>true</use_sim_time>
         <topic>cmd_vel</topic>
+        <odom_topic>odom</odom_topic>
+        <tf_topic>/tf</tf_topic>
+        <frame_id>odom</frame_id>
+        <child_frame_id>base_link</child_frame_id>
     </plugin>
     <!-- Moving Forward with Arrow Key Control plugin -->
@@ -264,12 +263,13 @@
   <gazebo reference="imu_link"> <!-- imu_link has a more broad horizon-->
     <sensor type="gpu_ray" name="lidar_sensor">
+      <ignition_frame_id>imu_link</ignition_frame_id>
       <topic>/scan</topic>
       <pose>0 0 0 0 0 0</pose>
       <visualize>true</visualize>
-      <update_rate>200</update_rate>
+      <update_rate>20</update_rate>
       <ray>
         <scan>
           <horizontal>
-            <samples>50</samples> <!-- on my computer, number of rays and update rate should not be too much, otherwise computer freezes-->
+            <samples>100</samples> <!-- on my computer, number of rays and update rate should not be too much, otherwise computer freezes-->
             <resolution>1</resolution>
             <min_angle>-1.5708</min_angle>
@@ -277,8 +277,12 @@
           </horizontal>
           <vertical>
-            <samples>50</samples>
+            <!-- <samples>50</samples>
             <resolution>1</resolution>
             <min_angle>-1.5708</min_angle>
-            <max_angle>1.5708</max_angle>
+            <max_angle>1.5708</max_angle> -->
+            <samples>1</samples>
+            <resolution>1</resolution>
+            <min_angle>0</min_angle>
+            <max_angle>0</max_angle>
           </vertical>
         </scan>

Commit message: Fixed the Gazebo crash by recalculating the base_link inertia values. Added 2 new maps and lowered the map Z-offset to prevent the floor from clipping.

File: sentry_gazebo/urdf/test_robot.xacro (robot description, xacro)
@@ -4,9 +4,10 @@
   <xacro:property name="radius_wheel" value="0.06" />
   <xacro:property name="PI" value="3.1415926"/>
-  <xacro:macro name="default_inertial" params="mass">
+  <xacro:macro name="wheel_inertial" params="mass">
     <inertial>
       <mass value="${mass}" />
-      <inertia ixx="0.01" ixy="0.0" ixz="0.0"
-                    iyy="0.01" iyz="0.0" izz="0.01" />
+      <inertia ixx="0.00055" ixy="0.0" ixz="0.0"
+               iyy="0.00055" iyz="0.0"
+               izz="0.0009" />
     </inertial>
   </xacro:macro>
@@ -30,5 +31,10 @@
       <origin rpy="0 0 ${PI/2}" xyz="0 0 0.05"/>
     </collision>
-    <xacro:default_inertial mass="8.2"/>
+    <inertial>
+      <mass value="8.2"/>
+      <inertia ixx="0.0683" ixy="0" ixz="0"
+               iyy="0.0342" iyz="0"
+               izz="0.0888" />
+    </inertial>
   </link>
   <link name="wheel_1">
@@ -49,5 +55,5 @@
     <mu1>0.5</mu1>
     <mu2>0.5</mu2>
-    <xacro:default_inertial mass="0.5"/>
+    <xacro:wheel_inertial mass="0.5"/>
   </link>
   <link name="wheel_2">
@@ -66,5 +72,5 @@
     <mu1>0.5</mu1>
     <mu2>0.5</mu2>
-    <xacro:default_inertial mass="0.5"/>
+    <xacro:wheel_inertial mass="0.5"/>
   </link>
   <link name="wheel_3">
@@ -83,5 +89,5 @@
     <mu1>0.5</mu1>
     <mu2>0.5</mu2>
-    <xacro:default_inertial mass="0.5"/>
+    <xacro:wheel_inertial mass="0.5"/>
   </link>
   <link name="wheel_4">
@@ -100,5 +106,5 @@
     <mu1>0.5</mu1>
     <mu2>0.5</mu2>
-    <xacro:default_inertial mass="0.5"/>
+    <xacro:wheel_inertial mass="0.5"/>
   </link>
   <joint name="base_to_wheel1" type="continuous">
@@ -179,5 +185,5 @@
         <right_joint>base_to_wheel3</right_joint>
         <right_joint>base_to_wheel4</right_joint>
-        <wheel_separation>1.2</wheel_separation>
+        <wheel_separation>0.45</wheel_separation>
         <wheel_radius>${radius_wheel}</wheel_radius>
         <odom_publish_frequency>50</odom_publish_frequency>
@@ -271,5 +277,5 @@
         <scan>
           <horizontal>
-            <samples>100</samples> <!-- on my computer, number of rays and update rate should not be too much, otherwise computer freezes-->
+            <samples>360</samples> <!-- on my computer, number of rays and update rate should not be too much, otherwise computer freezes-->
             <resolution>1</resolution>
             <min_angle>-1.5708</min_angle>

Commit message: Added FAST-LIO mapping and drivers

File: sentry_gazebo/urdf/test_robot.xacro (robot description, xacro)
@@ -264,45 +264,39 @@
     </sensor>
   </gazebo>
-  <!-- LiDAR sensor -->
-  <!-- https://gazebosim.org/docs/fortress/sensors/#lidar-sensor -->
-  <!-- topic name in ign topic -l: /world/default/model/testbot/link/dummy/sensor/lidar_sensor/scan -->
-  <gazebo reference="imu_link"> <!-- imu_link has a more broad horizon-->
-    <sensor type="gpu_ray" name="lidar_sensor">
+  <gazebo reference="imu_link">
+    <sensor type="gpu_lidar" name="livox_mid360">
       <ignition_frame_id>imu_link</ignition_frame_id>
-      <topic>/scan</topic>
+      <topic>/lidar_points</topic>
       <pose>0 0 0 0 0 0</pose>
       <visualize>true</visualize>
-      <update_rate>20</update_rate>
-      <ray>
+      <update_rate>10</update_rate>
+      <always_on>true</always_on>
+      <lidar>
         <scan>
           <horizontal>
-            <samples>360</samples> <!-- on my computer, number of rays and update rate should not be too much, otherwise computer freezes-->
-            <resolution>1</resolution>
-            <min_angle>-1.5708</min_angle>
-            <max_angle>1.5708</max_angle>
+            <samples>2000</samples>
+            <resolution>1.0</resolution>
+            <min_angle>-${PI}</min_angle>
+            <max_angle>${PI}</max_angle>
           </horizontal>
           <vertical>
-            <!-- <samples>50</samples>
-            <resolution>1</resolution>
-            <min_angle>-1.5708</min_angle>
-            <max_angle>1.5708</max_angle> -->
-            <samples>1</samples>
-            <resolution>1</resolution>
-            <min_angle>0</min_angle>
-            <max_angle>0</max_angle>
+            <samples>100</samples>
+            <resolution>1.0</resolution>
+            <min_angle>-0.515</min_angle>
+            <max_angle>0.515</max_angle>
           </vertical>
         </scan>
         <range>
-          <min>0.2</min>
-          <max>10.0</max>
+          <min>0.05</min>
+          <max>70.0</max>
           <resolution>0.01</resolution>
         </range>
-      </ray>
+        <noise>
+          <type>gaussian</type>
+          <mean>0.0</mean>
+          <stddev>0.02</stddev>
+        </noise>
+      </lidar>
     </sensor>
   </gazebo>
-  <!-- Livox-Mid360  -->
-  <!--<xacro:include filename="$(find ros2_livox_simulation)/urdf/mid360.xacro" />
-  <xacro:mid360 name="livox_frame" parent="base_link" topic="/livox/lidar">
-    <origin xyz="$(arg xyz)" rpy="$(arg rpy)" />
-  </xacro:mid360> -->
 </robot>
